Commit message: ugh i hate gripping

File: catkin_ws/src/robot/ur5/ur5_description/urdf/ur5.urdf.xacro (robot description, xacro)
@@ -265,9 +265,9 @@
         </material>
       </visual>
-      <collision>
+      <!-- <collision>
         <geometry>
           <mesh filename="package://ur5_description/meshes/ur5/collision/wrist3.stl" />
         </geometry>
-      </collision>
+      </collision> -->
       <xacro:cylinder_inertial radius="0.6" length="0.12" mass="${wrist_3_mass}">
         <origin xyz="0.0 0.0 0.0" rpy="0 0 0" />
@@ -280,10 +280,10 @@
     </joint>
     <link name="${prefix}ee_link">
-      <collision>
+      <!-- <collision>
         <geometry>
           <box size="0.01 0.01 0.01"/>
         </geometry>
         <origin rpy="0 0 0" xyz="-0.01 0 0"/>
-      </collision>
+      </collision> -->
     </link>
     <xacro:ur_arm_transmission prefix="${prefix}" />

File: catkin_ws/src/robot/ur5/ur5_description/urdf/ur5_robotiq85_gripper.urdf.xacro (robot description, xacro)
@@ -14,9 +14,9 @@
       <material name="flat_black"/>
     </visual>
-    <collision>
+    <!-- <collision>
       <geometry>
         <mesh filename="package://robotiq_description/meshes/robotiq_85_coupler.stl" />
       </geometry>
-    </collision>
+    </collision> -->
     <inertial>
       <origin xyz="2.073e-05   1.45286e-03  -1.1049e-03" rpy="0 0 0" />
@@ -65,5 +65,5 @@
         <attach_steps>2</attach_steps>    <!-- default: 20 -->
         <detach_steps>2</detach_steps>    <!-- default: 40 -->
-        <min_contact_count>3</min_contact_count>
+        <min_contact_count>1</min_contact_count>
       </grasp_check>
       <gripper_link>robotiq_85_left_finger_tip_link</gripper_link>
